File: DACAmps.sch (KiCad schematic (older format))
At the start: 15 parts, among them IC26 TDA2822D013TR

Commit message: Checkpoint before trying 4 layer
Parts:
- IC26: footprint SOIC127P600X175-8N -> Package_SO:SOIC-8_3.9x4.9mm_P1.27mm
Changed lines of the file:
@@
 $Descr A4 11693 8268
 encoding utf-8
-Sheet 41 50
+Sheet 41 51
 Title ""
 Date ""
@@
 F 0 "IC26" H 5850 3915 50  0000 C CNN
 F 1 "TDA2822D013TR" H 5850 3824 50  0000 C CNN
-F 2 "SOIC127P600X175-8N" H 6700 3750 50  0001 L CNN
+F 2 "Package_SO:SOIC-8_3.9x4.9mm_P1.27mm" H 6700 3750 50  0001 L CNN
 F 3 "https://www.st.com/resource/en/datasheet/tda2822d.pdf" H 6700 3650 50  0001 L CNN
 F 4 "STMICROELECTRONICS - TDA2822D013TR - Audio Power Amplifier, 300 mW, AB, 2 Channel, 1.8V to 15V, SOIC, 8 Pins" H 6700 3550 50  0001 L CNN "Description"
