File: PWM.sch (KiCad schematic (older format))
At the start: 2 parts, among them IC21 FAN3122TMX

Commit message: Checkpoint before trying 4 layer
Parts:
- IC21: footprint SOIC127P600X175-8N -> Package_SO:SOIC-8_3.9x4.9mm_P1.27mm
Changed lines of the file:
@@
 $Descr A4 11693 8268
 encoding utf-8
-Sheet 38 50
+Sheet 34 44
 Title ""
 Date ""
@@
 AR Path="/60F2EF44/60F295A7" Ref="IC22"  Part="1"
 AR Path="/60F327BB/60F295A7" Ref="IC23"  Part="1"
-F 0 "IC23" H 5800 3865 50  0000 C CNN
+F 0 "IC21" H 5800 3865 50  0000 C CNN
 F 1 "FAN3122TMX" H 5800 3774 50  0000 C CNN
-F 2 "SOIC127P600X175-8N" H 6250 3700 50  0001 L CNN
+F 2 "Package_SO:SOIC-8_3.9x4.9mm_P1.27mm" H 6250 3700 50  0001 L CNN
 F 3 "http://www.onsemi.com/pub/Collateral/FAN3122T_F085-D.PDF" H 6250 3600 50  0001 L CNN
 F 4 "TTL input, single non-inverting output, peak 11.4A sink, 10.6A source current Low-Side Gate Driver" H 6250 3500 50  0001 L CNN "Description"
@@
 AR Path="/60F2EF44/60F2B2A2" Ref="C60"  Part="1"
 AR Path="/60F327BB/60F2B2A2" Ref="C61"  Part="1"
-F 0 "C61" H 5915 2996 50  0000 L CNN
+F 0 "C59" H 5915 2996 50  0000 L CNN
 F 1 "1uF" H 5915 2905 50  0000 L CNN
 F 2 "Capacitor_SMD:C_0805_2012Metric" H 5838 2800 50  0001 C CNN
