File: Power Supply.sch (KiCad schematic (older format))
At the start: 15 parts, among them IC1 XL1509-5.0E1, U1 AMS1117-3.3

Commit message: Checkpoint before trying 4 layer
Parts:
- IC1: footprint SOIC127P600X175-8N -> Package_SO:SOIC-8-1EP_3.9x4.9mm_P1.27mm_EP2.29x3mm
- L1: footprint INDPM125125X800N -> Inductor_SMD:L_12x12mm_H6mm
Changed lines of the file:
@@
 $Descr A4 11693 8268
 encoding utf-8
-Sheet 2 50
+Sheet 2 52
 Title ""
 Date ""
@@
 F 0 "IC1" H 4750 2465 50  0000 C CNN
 F 1 "XL1509-5.0E1" H 4750 2374 50  0000 C CNN
-F 2 "SOIC127P600X175-8N" H 5100 2300 50  0001 L CNN
+F 2 "Package_SO:SOIC-8-1EP_3.9x4.9mm_P1.27mm_EP2.29x3mm" H 5100 2300 50  0001 L CNN
 F 3 "https://datasheet.lcsc.com/szlcsc/XLSEMI-XL1509-5-0E1_C61063.pdf" H 5100 2200 50  0001 L CNN
 F 4 "2A 150KHz 40V Buck DC to DC Converter." H 5100 2100 50  0001 L CNN "Description"
@@
 F 0 "L1" H 7050 2225 50  0000 C CNN
 F 1 "SWRB1207S-680MT" H 7050 2134 50  0000 C CNN
-F 2 "INDPM125125X800N" H 7300 2050 50  0001 L CNN
+F 2 "Inductor_SMD:L_12x12mm_H6mm" H 7300 2050 50  0001 L CNN
 F 3 "https://datasheet.lcsc.com/szlcsc/Sunlord-SWRB1207S-680MT_C169377.pdf" H 7300 1950 50  0001 L CNN
 F 4 "Power Inductors 68uH +/-20% 2.1A SMD,12.5x12.5x8mm(max) RoHS" H 7300 1850 50  0001 L CNN "Description"
