File: EEPROM.sch (KiCad schematic (older format))
At the start: 4 parts, among them IC2 M24M02-DRMN6TP

Commit message: Routed PCB
Parts:
- C29: JLCPCB_PN (none) -> C49678
- IC2: JLCPCB_PN (none) -> C115042
- R21, R22: JLCPCB_PN (none) -> C17673
Changed lines of the file:
@@
 F 8 "STMicroelectronics" H 6200 3100 50  0001 L CNN "Manufacturer_Name"
 F 9 "M24M02-DRMN6TP" H 6200 3000 50  0001 L CNN "Manufacturer_Part_Number"
+F 10 "C115042" H 5250 3600 50  0001 C CNN "JLCPCB_PN"
 	1    5250 3600
 	1    0    0    -1
@@
 F 2 "Capacitor_SMD:C_0805_2012Metric" H 5850 2850 50  0001 C CNN
 F 3 "~" H 5850 2850 50  0001 C CNN
+F 4 "C49678" H 5850 2850 50  0001 C CNN "JLCPCB_PN"
 	1    5850 2850
 	0    1    1    0
@@
 F 2 "Resistor_SMD:R_0805_2012Metric" V 6890 3840 50  0001 C CNN
 F 3 "~" H 6850 3850 50  0001 C CNN
+F 4 "C17673" H 6850 3850 50  0001 C CNN "JLCPCB_PN"
 	1    6850 3850
 	0    1    1    0
@@
 F 2 "Resistor_SMD:R_0805_2012Metric" V 6840 4140 50  0001 C CNN
 F 3 "~" H 6800 4150 50  0001 C CNN
+F 4 "C17673" H 6800 4150 50  0001 C CNN "JLCPCB_PN"
 	1    6800 4150
 	0    1    1    0
