File: GearFeedback.sch (KiCad schematic (older format))
At the start: 9 parts

Commit message: Checkpoint before trying 4 layer
Connections:
- net 3_3Vcc: now also R23.1, R27.1
Changed lines of the file:
@@
 $Descr A4 11693 8268
 encoding utf-8
-Sheet 21 50
+Sheet 18 37
 Title ""
 Date ""
@@
 	4700 2600 4700 2200
 Wire Wire Line
-	4700 2200 6750 2200
-Wire Wire Line
 	6750 2200 6750 2550
 Wire Wire Line
-	5850 2600 5850 1800
+	5850 2600 5850 2200
 Wire Wire Line
 	4700 3150 4050 3150
@@
 Text HLabel 5800 5600 0    50   Input ~ 0
 GND
+Wire Wire Line
+	4700 2200 5850 2200
+Connection ~ 5850 2200
+Wire Wire Line
+	5850 2200 5850 1800
+Wire Wire Line
+	5850 2200 6750 2200
 $EndSCHEMATC

Commit message: Routed PCB
Parts:
- C30, C31, C32: JLCPCB_PN (none) -> C28323
- R23, R24, R25, R26, R27, R28: JLCPCB_PN (none) -> C17513
Changed lines of the file:
@@
 F 2 "Resistor_SMD:R_0805_2012Metric" V 4740 2740 50  0001 C CNN
 F 3 "~" H 4700 2750 50  0001 C CNN
+F 4 "C17513" H 4700 2750 50  0001 C CNN "JLCPCB_PN"
 	1    4700 2750
 	1    0    0    -1
@@
 F 2 "Resistor_SMD:R_0805_2012Metric" V 5890 2740 50  0001 C CNN
 F 3 "~" H 5850 2750 50  0001 C CNN
+F 4 "C17513" H 5850 2750 50  0001 C CNN "JLCPCB_PN"
 	1    5850 2750
 	1    0    0    -1
@@
 F 2 "Resistor_SMD:R_0805_2012Metric" V 6790 2690 50  0001 C CNN
 F 3 "~" H 6750 2700 50  0001 C CNN
+F 4 "C17513" H 6750 2700 50  0001 C CNN "JLCPCB_PN"
 	1    6750 2700
 	1    0    0    -1
@@
 F 2 "Resistor_SMD:R_0805_2012Metric" V 4740 3840 50  0001 C CNN
 F 3 "~" H 4700 3850 50  0001 C CNN
+F 4 "C17513" H 4700 3850 50  0001 C CNN "JLCPCB_PN"
 	1    4700 3850
 	1    0    0    -1
@@
 F 2 "Resistor_SMD:R_0805_2012Metric" V 5890 3790 50  0001 C CNN
 F 3 "~" H 5850 3800 50  0001 C CNN
+F 4 "C17513" H 5850 3800 50  0001 C CNN "JLCPCB_PN"
 	1    5850 3800
 	1    0    0    -1
@@
 F 2 "Resistor_SMD:R_0805_2012Metric" V 6790 3790 50  0001 C CNN
 F 3 "~" H 6750 3800 50  0001 C CNN
+F 4 "C17513" H 6750 3800 50  0001 C CNN "JLCPCB_PN"
 	1    6750 3800
 	1    0    0    -1
@@
 F 2 "Capacitor_SMD:C_0805_2012Metric" H 4700 4750 50  0001 C CNN
 F 3 "~" H 4700 4750 50  0001 C CNN
+F 4 "C28323" H 4700 4750 50  0001 C CNN "JLCPCB_PN"
 	1    4700 4750
 	1    0    0    -1
@@
 F 2 "Capacitor_SMD:C_0805_2012Metric" H 5850 4750 50  0001 C CNN
 F 3 "~" H 5850 4750 50  0001 C CNN
+F 4 "C28323" H 5850 4750 50  0001 C CNN "JLCPCB_PN"
 	1    5850 4750
 	1    0    0    -1
@@
 F 2 "Capacitor_SMD:C_0805_2012Metric" H 6750 4700 50  0001 C CNN
 F 3 "~" H 6750 4700 50  0001 C CNN
+F 4 "C28323" H 6750 4700 50  0001 C CNN "JLCPCB_PN"
 	1    6750 4700
 	1    0    0    -1
