File: HighSide12VSwitch.sch (KiCad schematic (older format))
At the start: 1 part, among them Q2 NCV8461DR2G

Commit message: Checkpoint before trying 4 layer
Changed lines of the file:
@@
 $Descr A4 11693 8268
 encoding utf-8
-Sheet 51 51
+Sheet 46 37
 Title ""
 Date ""
@@
 AR Path="/60458FBE/6045991B" Ref="Q2"  Part="1"
 AR Path="/61BFDF6F/6045991B" Ref="Q?"  Part="1"
-F 0 "Q?" H 5600 4065 50  0000 C CNN
+AR Path="/61C2C201/6045991B" Ref="Q6"  Part="1"
+F 0 "Q6" H 5600 4065 50  0000 C CNN
 F 1 "NCV8461DR2G" H 5600 3974 50  0000 C CNN
 F 2 "SamacSys_Parts:SOIC127P600X175-8N" H 6000 3900 50  0001 L CNN
@@
 AR Path="/60458FBE/6045A26D" Ref="#PWR085"  Part="1"
 AR Path="/61BFDF6F/6045A26D" Ref="#PWR?"  Part="1"
-F 0 "#PWR?" H 4800 3550 50  0001 C CNN
+AR Path="/61C2C201/6045A26D" Ref="#PWR0101"  Part="1"
+F 0 "#PWR0101" H 4800 3550 50  0001 C CNN
 F 1 "GND" V 4805 3672 50  0000 R CNN
 F 2 "" H 4800 3800 50  0001 C CNN

Commit message: Routed PCB
Parts:
- Q2: JLCPCB_PN (none) -> C154603
Changed lines of the file:
@@
 F 8 "ON Semiconductor" H 6000 3300 50  0001 L CNN "Manufacturer_Name"
 F 9 "NCV8461DR2G" H 6000 3200 50  0001 L CNN "Manufacturer_Part_Number"
+F 10 "C154603" H 5050 3800 50  0001 C CNN "JLCPCB_PN"
 	1    5050 3800
 	1    0    0    -1
