File: LinBUS.sch (KiCad schematic (older format))
At the start: 11 parts, among them IC12 TJA1020T_CM,118, Q5 MMBT3904

Commit message: Checkpoint before trying 4 layer
Parts:
- IC12: footprint SOIC127P600X175-8N -> Package_SO:SO-8_3.9x4.9mm_P1.27mm
Changed lines of the file:
@@
 $Descr A4 11693 8268
 encoding utf-8
-Sheet 29 50
+Sheet 22 37
 Title ""
 Date ""
@@
 F 0 "IC12" H 5650 4065 50  0000 C CNN
 F 1 "TJA1020T_CM,118" H 5650 3974 50  0000 C CNN
-F 2 "SOIC127P600X175-8N" H 6050 3900 50  0001 L CNN
+F 2 "Package_SO:SO-8_3.9x4.9mm_P1.27mm" H 6050 3900 50  0001 L CNN
 F 3 "http://www.nxp.com/docs/en/data-sheet/TJA1020.pdf" H 6050 3800 50  0001 L CNN
 F 4 "NXP - TJA1020T/CM,118 - LIN TRANSCEIVER, AUTO, 20KBAUD, SOIC8" H 6050 3700 50  0001 L CNN "Description"

Commit message: Routed PCB
Parts:
- C24: JLCPCB_PN (none) -> C53175
- C25: JLCPCB_PN (none) -> C28323
- D14: JLCPCB_PN (none) -> C81598
- IC12: JLCPCB_PN (none) -> C128810
- Q5: JLCPCB_PN (none) -> C20526
- R47: JLCPCB_PN (none) -> C17513
- R49: JLCPCB_PN (none) -> C17414
- R50, R53: JLCPCB_PN (none) -> C17520
- R51: value R_US -> 1K; JLCPCB_PN (none) -> C17513
- R54: JLCPCB_PN (none) -> C17506
Changed lines of the file:
@@
 F 8 "NXP" H 6050 3300 50  0001 L CNN "Manufacturer_Name"
 F 9 "TJA1020T/CM,118" H 6050 3200 50  0001 L CNN "Manufacturer_Part_Number"
+F 10 "C128810" H 5100 3800 50  0001 C CNN "JLCPCB_PN"
 	1    5100 3800
 	1    0    0    -1
@@
 F 2 "Resistor_SMD:R_0805_2012Metric" V 3690 3090 50  0001 C CNN
 F 3 "~" H 3650 3100 50  0001 C CNN
+F 4 "C17414" H 3650 3100 50  0001 C CNN "JLCPCB_PN"
 	1    3650 3100
 	1    0    0    -1
@@
 F 2 "Resistor_SMD:R_0805_2012Metric" V 4190 3090 50  0001 C CNN
 F 3 "~" H 4150 3100 50  0001 C CNN
+F 4 "C17520" H 4150 3100 50  0001 C CNN "JLCPCB_PN"
 	1    4150 3100
 	1    0    0    -1
@@
 F 2 "Resistor_SMD:R_0805_2012Metric" V 4640 3090 50  0001 C CNN
 F 3 "~" H 4600 3100 50  0001 C CNN
+F 4 "C17520" H 4600 3100 50  0001 C CNN "JLCPCB_PN"
 	1    4600 3100
 	1    0    0    -1
@@
 F 2 "Resistor_SMD:R_0805_2012Metric" V 7390 3740 50  0001 C CNN
 F 3 "~" H 7350 3750 50  0001 C CNN
+F 4 "C17506" H 7350 3750 50  0001 C CNN "JLCPCB_PN"
 	1    7350 3750
 	1    0    0    -1
@@
 P 4250 4000
 F 0 "R51" H 4318 4046 50  0000 L CNN
-F 1 "R_US" H 4318 3955 50  0000 L CNN
+F 1 "1K" H 4318 3955 50  0000 L CNN
 F 2 "Resistor_SMD:R_0805_2012Metric" V 4290 3990 50  0001 C CNN
 F 3 "~" H 4250 4000 50  0001 C CNN
+F 4 "C17513" H 4250 4000 50  0001 C CNN "JLCPCB_PN"
 	1    4250 4000
 	0    -1   -1   0
@@
 F 2 "Resistor_SMD:R_0805_2012Metric" V 2690 5140 50  0001 C CNN
 F 3 "~" H 2650 5150 50  0001 C CNN
+F 4 "C17513" H 2650 5150 50  0001 C CNN "JLCPCB_PN"
 	1    2650 5150
 	0    -1   -1   0
@@
 F 2 "Package_TO_SOT_SMD:SOT-23" H 3650 5075 50  0001 L CIN
 F 3 "https://www.fairchildsemi.com/datasheets/2N/2N3904.pdf" H 3450 5150 50  0001 L CNN
+F 4 "C20526" H 3450 5150 50  0001 C CNN "JLCPCB_PN"
 	1    3450 5150
 	1    0    0    -1
@@
 F 11 "Diodes Incorporated" H 7550 4200 60  0001 L CNN "Manufacturer"
 F 12 "Active" H 7550 4300 60  0001 L CNN "Status"
+F 13 "C81598" H 7350 3100 50  0001 C CNN "JLCPCB_PN"
 	1    7350 3100
 	0    1    1    0
@@
 F 2 "Capacitor_SMD:C_0805_2012Metric" H 7900 2600 50  0001 C CNN
 F 3 "~" H 7900 2600 50  0001 C CNN
+F 4 "C28323" H 7900 2600 50  0001 C CNN "JLCPCB_PN"
 	1    7900 2600
 	0    -1   -1   0
@@
 F 2 "Capacitor_SMD:C_0805_2012Metric" H 7350 4600 50  0001 C CNN
 F 3 "~" H 7350 4600 50  0001 C CNN
+F 4 "C53175" H 7350 4600 50  0001 C CNN "JLCPCB_PN"
 	1    7350 4600
 	1    0    0    -1
