File: MS43Zombie.sch (KiCad schematic (older format))
At the start: 7 parts, among them J1 7-967288-1, J6 X62102, J7 X62202, J8 X62101, J9 X62201

Commit message: Checkpoint before trying 4 layer
Parts:
- added J2: EXT1, Connector_PinHeader_2.54mm:PinHeader_2x20_P2.54mm_Vertical, symbol Connector_Generic:Conn_02x20_Odd_Even
- added J4: EXT2, Connector_PinHeader_2.54mm:PinHeader_2x20_P2.54mm_Vertical, symbol Connector_Generic:Conn_02x20_Odd_Even
Connections:
- net labels added: 12V_MEASURE, CAN_EXT2+, CAN_EXT2-, COOLANT_PUMP_1, COOLANT_PUMP_2, CoolantTempIn, FuelPumpRelayDRV, LED, PA4, PA5, PA6, PA7, PB0, PB12, PB13, PB14, PB15, PB7, PD13, PD14, PD15, PD4, PD5, PD8, PD9, PE0, PE1, PE10, PE11, PE12, PE13, PE14, PE15, PWMCoolantPump1, PWMCoolantPump2, RST, RTC_TAMPER, ReverseLightRelay, ReverseRelayDRV, SignalShiftLock, SteptronicTipDown, SteptronicTipUp, SupplyShiftLock, VBAT, VREF+, VREF-, WKUP
- net labels removed: +12Vin, CAN3_EXTH, CAN3_EXTL, CAN3_INT, CAN3_SBY, CAN_EXT2H, CAN_EXT2L, CAN_EXT3H, CAN_EXT3L, CharacteristicMapCoolingThermostat, DAC1, DAC2, ElectricThrottleBodyActuator1, ElectricThrottleBodyActuator2, GP12V_IN, GP1_DRV, GP2_DRV, GP3_DRV, GP_OUT1, GP_OUT2, GP_OUT3, GroundElectricThrottleBody, GroundExhaustCamshaftSensor, GroundIntakeCamshaft, GroundMAF, HVREQ_IN, HeaterEnable, HeaterNTCSignal, HeaterNTCSupply, INVERTER_POWER, IdleSpeedActuatorClosing, IdleSpeedActuatorOpening, MAIN_DRV, PCH_DRV, PWM1, PWM2, PWM3, RS232_RX, RS232_TX, SPI2_MISO, SPI2_MOSI, SPI2_NSS, SPI2_SCK, SW_MODE0, SW_MODE1, ShieldKnockSensors, SignalElectricThrottleBodyPot2, SignalExhaustCamshaftSensor, SignalFuelTankVentValve, SignalMAF, SignalSecondaryAirPumpValve, SignalVANOSExhaustSolenoid, SignalVANOSIntakeSolenoid, VariableIntakeManifoldFlap
- wire segments 168 -> 156
- no-connect marks 70 -> 103
Other:
- note removed: "8 pins"

Commit message: 4 layer board that passes checks
Parts:
- removed F2: 20A, symbol Device:Fuse
- removed F4: 30A, symbol Device:Fuse
- added D1: SS54B, DIOM5336X244N, symbol SamacSys_Parts:SS54B
Connections:
- net labels added: ACCompressorRelayDRV, DigitalPotA1, DigitalPotA2, DigitalPotW1, DigitalPotW2, FuelInjectorDRV, MG1_TEMP_IN, MG2_TEMP_IN, PC10, PC11, PD10, PD11, UART4_RX, UART4_TX, USB_VBUS_ON
- net labels removed: POT1_CS, POT1_OUT, POT2_CS, POT2_OUT, SPI3_MOSI, SPI3_SCK, USART1_RX, USART1_TX
- wire segments 156 -> 185
- no-connect marks 103 -> 100

Commit message: Routed PCB
Parts:
- D1: JLCPCB_PN (none) -> C22452
Changed lines of the file:
@@
 F 8 "HY Electronic Corp" H 5200 8400 50  0001 L CNN "Manufacturer_Name"
 F 9 "SS54B" H 5200 8300 50  0001 L CNN "Manufacturer_Part_Number"
+F 10 "C22452" H 4750 9000 50  0001 C CNN "JLCPCB_PN"
 	1    4750 9000
 	1    0    0    1

Commit message: Checkpoint 2022-01-19
Design with bluepill to run the heater since we lose some of the SPI
pins to the USB port on the STM32-H107.
Parts:
- added U1: YAAJ_BluePill, Footprints:YAAJ_BluePill_1, symbol YAAJ_BluePill:YAAJ_BluePill
- D1: footprint DIOM5336X244N -> SamacSys_Parts:DIOM5336X244N
Connections:
- net PA7 is gone; now on net LIN_NSLP: J4.25 (Pin_25)
- net PC4 is gone; now on net MG2_TEMP_IN: J4.19 (Pin_19)
- net PC5 is gone; now on net MG1_TEMP_IN: J4.18 (Pin_18)
- net 3_3Vcc: now also U1.20 (3V3), U1.38 (3V3)
- net 5Vcc: now also U1.18 (5V)
- net GNDPWR: now also U1.19 (GND), U1.39 (GND), U1.40 (GND)
- net LIN_NSLP: no longer J4.28 (Pin_28)
- net MG1_TEMP_IN: no longer J2.12 (Pin_12)
- net MG2_TEMP_IN: no longer J2.11 (Pin_11)
- net IHKA_DEMAND_IN: now reaches J1.C3
- net IHKA_DEMAND_IN: now also U1.6 (PA9)
- net PA8: now reaches J4.24 (Pin_24)
- net PD2: now reaches J4.6 (Pin_6)
- net PD2: now also U1.28 (PA3)
- net PD3: now reaches J4.7 (Pin_7)
- net PD3: now also U1.7 (PA10)
- net REV_IN renamed PC12
- net PC12: now also U1.27 (PA2)
- net SCL renamed PB8
- net SDA renamed PB9
- net SL1- renamed PC9
- net SL2- renamed PC8
- net SP renamed PD12
- net T15_IN renamed PD6
- net UART3_RX renamed PB11
- net UART3_TX renamed PB10
- net USART2_CLK renamed PA1
- net USART2_REQ renamed PE6
- net USART2_RX renamed PA3
- net USART2_TX renamed PA2
- new net ERROR_LIGHT: U1.11 (PB3)
- new net EXTRA_TEMP: U1.30 (PA5)
- new net HEATER_CONTACTOR: U1.1 (PB12)
- new net HEATER_PUMP_ENABLE: U1.2 (PB13)
- new net PA4: J4.28 (Pin_28)
- new net PE12: J2.11 (Pin_11)
- new net PE13: J2.12 (Pin_12)
- new net SWCAN_MODE0: U1.15 (PB7)
- new net SWCAN_MODE1: U1.14 (PB6)
- new net SWCAN_RX: U1.16 (PB8)
- new net SWCAN_TX: U1.17 (PB9)
- new net WATER_PUMP_PWM: U1.31 (PA6)
- new net WATER_TEMP: U1.29 (PA4)
- no-connect marks 100 -> 123
