File: MTH.sch (KiCad schematic (older format))
At the start: 3 parts, among them U19 SN65HVD230

Commit message: Routed PCB
Parts:
- C66: JLCPCB_PN (none) -> C49678
- R78: JLCPCB_PN (none) -> C17437
- U19: JLCPCB_PN (none) -> C12084
Changed lines of the file:
@@
 $Descr A4 11693 8268
 encoding utf-8
-Sheet 20 36
+Sheet 16 36
 Title ""
 Date ""
@@
 F 2 "Package_SO:SOIC-8_3.9x4.9mm_P1.27mm" H 5850 3000 50  0001 C CNN
 F 3 "http://www.ti.com/lit/ds/symlink/sn65hvd230.pdf" H 5750 3900 50  0001 C CNN
+F 4 "C12084" H 5850 3500 50  0001 C CNN "JLCPCB_PN"
 	1    5850 3500
 	1    0    0    -1
@@
 F 2 "Resistor_SMD:R_0805_2012Metric" V 6840 3640 50  0001 C CNN
 F 3 "~" H 6800 3650 50  0001 C CNN
+F 4 "C17437" H 6800 3650 50  0001 C CNN "JLCPCB_PN"
 	1    6800 3650
 	1    0    0    -1
@@
 F 2 "Capacitor_SMD:C_0805_2012Metric" H 5850 2750 50  0001 C CNN
 F 3 "~" H 5850 2750 50  0001 C CNN
+F 4 "C49678" H 5850 2750 50  0001 C CNN "JLCPCB_PN"
 	1    5850 2750
 	-1   0    0    1
