File: Wifi.sch (KiCad schematic (older format))
At the start: 3 parts, among them J3 75867-101LF

Commit message: Routed PCB
Parts:
- C28: JLCPCB_PN (none) -> C15850
- FB1: JLCPCB_PN (none) -> C1015
Changed lines of the file:
@@
 $Descr A4 11693 8268
 encoding utf-8
-Sheet 8 36
+Sheet 7 36
 Title ""
 Date ""
@@
 F 8 "Bourns" H 4900 2400 50  0001 L CNN "Manufacturer_Name"
 F 9 "MH2029-300Y" H 4900 2300 50  0001 L CNN "Manufacturer_Part_Number"
+F 10 "C1015" H 4250 2900 50  0001 C CNN "JLCPCB_PN"
 	1    4250 2900
 	0    -1   -1   0
@@
 F 2 "Capacitor_SMD:C_0805_2012Metric" H 4800 3400 50  0001 C CNN
 F 3 "~" H 4800 3400 50  0001 C CNN
+F 4 "C15850" H 4800 3400 50  0001 C CNN "JLCPCB_PN"
 	1    4800 3400
 	1    0    0    -1
